Commit message: debug

File: XRoboToolkit-Teleop-Sample-Python/assets/piper/daul_piper.urdf (robot description, URDF)
Before this commit: robot bimanual_piper, 23 links, 22 joints
Joints:
- joint world_to_left_base: origin xyz=0 0.3 0 rpy=0 0 0 -> xyz=0 0.34 0 rpy=0 0 0
- joint world_to_right_base: origin xyz=0 -0.3 0 rpy=0 0 0 -> xyz=0 -0.34 0 rpy=0 0 0

File: piper_sdk/urdf/piper_description_d405.urdf (robot description, URDF)
Before this commit: robot piper, 12 links, 11 joints
Links:
- link base_link: geometry collision mesh filename=meshes/base_link.STL; visual mesh filename=meshes/base_link.STL
- link gripper_base: geometry collision mesh filename=meshes/gripper_base.STL; visual mesh filename=meshes/gripper_base.STL
- link link1: geometry collision mesh filename=meshes/link1.STL; visual mesh filename=meshes/link1.STL
- link link2: geometry collision mesh filename=meshes/link2.STL; visual mesh filename=meshes/link2.STL
- link link3: geometry collision mesh filename=meshes/link3.STL; visual mesh filename=meshes/link3.STL
- link link4: geometry collision mesh filename=meshes/link4.STL; visual mesh filename=meshes/link4.STL
- link link5: geometry collision mesh filename=meshes/link5.STL; visual mesh filename=meshes/link5.STL
- link link6: geometry collision mesh filename=meshes/link6.STL; visual mesh filename=meshes/link6.STL
- link link7: geometry collision mesh filename=meshes/link7.STL; visual mesh filename=meshes/link7.STL
- link link8: geometry collision mesh filename=meshes/link8.STL; visual mesh filename=meshes/link8.STL
- link link_cam: geometry collision mesh filename=meshes/camera.STL; visual mesh filename=meshes/camera.STL
